File: HPF_test_01/HPF_test_01.kicad_pcb (KiCad board)
At the start: 2 copper layers, 78.2 x 29.2 mm, 12 parts, among them T1 GT07-110-013

Commit message: Added hpf_freeCAD & STL files
Parts:
- moved T1 2.79 mm to (112.8, 92.5)
- moved TVS 2.79 mm to (113.8, 80.5)
- moved C2 0.51 mm to (107.4, 82.2)
Routing:
- net Net-(C1-Pad2): track 5.58 -> 7.60 mm
- net Net-(J2_BLACK1-Pad1): track 58.6 -> 56.6 mm
- net Net-(C2-Pad1): track 44.5 -> 46.1 mm
Other:
- outline, holes or cut-outs redrawn
- board text added: "HPF rev.02 feb2022 //keyudits"
- board text removed: "HPF rev.01 jan2022 //keyudits"
- board text removed: "non-plated cutout"

Commit message: moved to kicad 6.0
includes minor revision to board layout, increase clearance between TVS & C1
Parts:
- moved C2 2.69 mm to (105.2, 80.8)
- moved TVS 2.29 mm to (111.5, 80.5)
Routing:
- net Net-(C2-Pad2): track 20.7 -> 14.7 mm
Other:
- net class Default removed
- board text added: "HPF rev.03 june2022 //keyudits"
- board text removed: "HPF rev.02 feb2022 //keyudits"
