File: Plucker/plucker_v03/plucker_v03.kicad_sch (KiCad schematic)
At the start: 12 parts, among them J1_BNC1 BNC5-J-P-GN-RA-BH2D, J2_BLACK1 Conn_01x01, J3_RED1 Conn_01x01, T1 GT07-110-013, U1 SL1002A600SP

Commit message: assembled v03, added waveforms
Connections:
- net in: now reaches J3_RED1.1 (Pin_1), R1.1, RV1.2, V1.2 (E2)
Changed lines of the file:
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@@
   (junction (at 189.23 101.6) (diameter 0) (color 0 0 0 0)
+  )
+  (junction (at 84.455 129.54) (diameter 0) (color 0 0 0 0)
   )
   (junction (at 199.39 101.6) (diameter 0) (color 0 0 0 0)
@@
     (stroke (width 0) (type default) (color 0 0 0 0))
   )
+  (wire (pts (xy 84.455 129.54) (xy 84.455 133.35))
+    (stroke (width 0) (type default) (color 0 0 0 0))
+  )
   (wire (pts (xy 76.2 91.44) (xy 80.01 91.44))
     (stroke (width 0) (type default) (color 0 0 0 0))
@@
     (stroke (width 0) (type default) (color 0 0 0 0))
   )
-  (wire (pts (xy 80.01 129.54) (xy 94.615 129.54))
+  (wire (pts (xy 84.455 129.54) (xy 94.615 129.54))
+    (stroke (width 0) (type default) (color 0 0 0 0))
+  )
+  (wire (pts (xy 80.01 129.54) (xy 84.455 129.54))
     (stroke (width 0) (type default) (color 0 0 0 0))
   )
@@
     )
   )
+  (global_label "in" (shape input) (at 84.455 133.35 0) (fields_autoplaced)
+    (effects (font (size 1.27 1.27)) (justify left))
+    (property "Intersheet References" "${INTERSHEET_REFS}" (id 0) (at 88.533 133.2706 0)
+      (effects (font (size 1.27 1.27)) (justify left) hide)
+    )
+  )
